File: NFCCartridge.kicad_pcb (KiCad board)
At the start: 2 copper layers, 64.8 x 55.9 mm, 10 parts, among them J1 Cartridge Connector, U1 W25Q128, U2 ST25DVxxx

Commit message: Fixed error in cartridge connector pin assignments
Updated to version 1.2
Connections:
- J1 pad 1: GND -> +3V3
- J1 pad 2: +3V3 -> GND
- J1 pad 3: F_HOLD -> F_CS
- J1 pad 39: +5V -> +BATT
- J1 pad 4: F_CS -> F_HOLD
- J1 pad 40: +BATT -> +5V
- J1 pad 5: F_SCK -> F_MISO
- J1 pad 6: F_MISO -> F_SCK
- J1 pad 7: F_MOSI -> F_WP
- J1 pad 8: F_WP -> F_MOSI
Routing:
- net +3V3: track 45.9 -> 57.0 mm
- net F_CS: track 5.76 -> 9.51 mm
- net F_WP: track 11.1 -> 14.7 mm
- net F_MISO: track 8.82 -> 12.3 mm
- net F_MOSI: track 21.2 -> 18.7 mm
- net F_SCK: track 18.8 -> 16.3 mm
- net F_HOLD: track 13.9 -> 11.4 mm
Other:
- board text added: "v1.2"
